File: KiCAD/V1/Home sensor ESP32/Home sensor ESP32.kicad_sch (KiCad schematic)
At the start: 25 parts, among them J2 Conn_01x02_Socket, J3 Conn_01x04_Pin, J4 Conn_01x06_Socket, J5 Conn_01x08_Pin, J6 Conn_01x04_Pin, Q1 SI2312, Q2 SI2312, SW1 SW_SPDT, U1 ESP32-WROOM-32, U2 XC6210B332MR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

Commit message: .
Parts:
- R2, R3: value R -> 1K5
- R6, R7: value R -> 10k
Changed lines of the file:
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@@
 			)
 		)
-		(property "Value" "R"
+		(property "Value" "10k"
 			(at 80.01 142.24 90)
 			(effects
@@
 			)
 		)
-		(property "Value" "R"
+		(property "Value" "1K5"
 			(at 87.63 29.2099 0)
 			(effects
@@
 			)
 		)
-		(property "Value" "R"
+		(property "Value" "10k"
 			(at 80.01 124.46 90)
 			(effects
@@
 			)
 		)
-		(property "Value" "R"
+		(property "Value" "1K5"
 			(at 78.74 29.2099 0)
 			(effects
