File: KiCAD/V3/home sensor/home sensor.kicad_sch (KiCad schematic)
At the start: 48 parts, among them J1 USB_C_Receptacle_USB2.0_14P, J2 Conn_01x24_Socket, J3 Conn_01x02_Socket, J4 Conn_01x04_Socket, Q1 SI2312, Q2 SI2312, Q3 SI2312, U1 TP4056-42-ESOP8, U2 CP2102N-Axx-xQFN28, U3 ESP32-C6-MINI-1

Commit message: .
Parts:
- added C22, C23, C24, C25: 100nF, Capacitor_SMD:C_0805_2012Metric_Pad1.18x1.45mm_HandSolder, symbol Device:C
- added TP1, TP2, TP3, TP4: TestPoint, TestPoint:TestPoint_Pad_D1.5mm, symbol Connector:TestPoint
- added TP5: TestPoint, TestPoint:TestPoint_Bridge_Pitch2.54mm_Drill0.7mm, symbol Connector:TestPoint
- added U5: XC6210B332MR, Package_TO_SOT_SMD:SOT-23-5, symbol Regulator_Linear:XC6210B332MR
- J1: footprint Connector_USB:USB_C_Receptacle_Molex_105450-0101 -> Connector_USB:USB_C_Receptacle_G-Switch_GT-USB-7010ASV_model
- J4: footprint Connector_JST:JST_XH_B4B-XH-A_1x04_P2.50mm_Vertical -> Connector_PinSocket_2.54mm:PinSocket_1x04_P2.54mm_Horizontal
Connections:
- net +3.3V: now also J4.4 (Pin_4), C24.1, C25.1, TP4.1, U5.5 (VOUT)
- net BUSY: now also U3.29 (IO23)
- net CS: now also U3.24 (IO18)
- net DC: now also U3.27 (IO21)
- net GND: now also J4.3 (Pin_3), C22.2, C23.2, C24.2, C25.2, TP5.1, U5.2 (GND)
- net GPIO8: now also TP1.1
- net MOSI: now also U3.26 (IO20)
- net RESET: now also U3.28 (IO22)
- net SCK: now also U3.25 (IO19)
- net SCL: now also J4.2 (Pin_2)
- net SDA: now also J4.1 (Pin_1)
- net VBUS: now also TP3.1
- net at J3.1 (Pin_1), U1.5 (BAT): now also TP2.1
- new net +BATT: C22.1, C23.1, U5.1 (VIN), U5.3 (CE)
- no-connect marks 21 -> 30
Other:
- moved on the sheet: J4
